Commit message: test on uv

File: description/depth_camera.xacro (robot description, xacro)
@@ -4,13 +4,7 @@
         <parent link="chassis" />
         <child link="camera_link" />
-        <origin xyz="${length+0.005} 0 ${height/2}" rpy="0 0 0" />
+        <origin xyz="${3/4 * length} 0 ${height + 0.5}" rpy="0 0 0" />
     </joint>
     <link name="camera_link">
-        <visual>
-            <geometry>
-                <box size="0.010 0.03 0.03"/>
-            </geometry>
-            <material name="red"/>
-        </visual>
     </link>
     <joint name="camera_optical_joint" type="fixed">
@@ -25,11 +19,11 @@
             <pose> 0 0 0 0 0 0 </pose>
             <visualize>true</visualize>
-            <update_rate>10</update_rate>
+            <update_rate>5</update_rate>
             <camera>
-                <horizontal_fov>1.089</horizontal_fov>
+                <horizontal_fov>1.85</horizontal_fov>
                 <image>
                     <format>B8G8R8</format>
                     <width>640</width>
-                    <height>480</height>
+                    <height>200</height>
                 </image>
                 <clip>
@@ -40,5 +34,5 @@
             <plugin name="camera_controller" filename="libgazebo_ros_camera.so">
                 <frame_name>camera_link_optical</frame_name>
-                <min_depth>0.1</min_depth>
+                <min_depth>0.001</min_depth>
                 <max_depth>100.0</max_depth>
             </plugin>

File: description/light.xacro (robot description, xacro)
@@ -44,12 +44,26 @@
             </spot>
         </light>
-        <plugin name='light_control' filename='libFlashLightPlugin.so'>
-            <enable>true</enable>
-            <light>
-                <id>neon_light</id>
-                <duration>0.5</duration>
-                <interval>0.5</interval>
-            </light>
-        </plugin>
+ <!--        <sensor name="light_camera" type="depth">
+            <pose>${1/2* length} 0 ${height + 0.5} ${-pi/2} 0 ${-pi/2}</pose>
+            <visualize>true</visualize>
+            <update_rate>5</update_rate>
+            <camera>
+                <horizontal_fov>1.85</horizontal_fov>
+                <image>
+                    <format>B8G8R8</format>
+                    <width>640</width>
+                    <height>1000</height>
+                </image>
+                <clip>
+                    <near>0.05</near>
+                    <far>8.0</far>
+                </clip>
+            </camera>
+            <plugin name="camera_controller" filename="libgazebo_ros_camera.so">
+                <frame_name>light_link</frame_name>
+                <min_depth>0.1</min_depth>
+                <max_depth>100.0</max_depth>
+            </plugin>
+        </sensor> -->
     </gazebo>
 </robot>
