Commit message: multiple lidar

File: description/lidar_3d.xacro (robot description, xacro)
@@ -1,47 +1,21 @@
 <?xml version="1.0"?>
 <robot xmlns:xacro="http://www.ros.org/wiki/xacro" name="robot">
-    <joint name="laser_3d_joint" type="fixed">
-        <parent link="chassis" />
-        <child link="laser_3d_frame" />
-        <origin xyz="${3/4 * length} 0 ${height + 0.5}" rpy="0 0 0" />
-    </joint>
-    <link name="laser_3d_frame">
-    </link>
-    <gazebo reference="laser_3d_frame">
-        <material>Gazebo/Red</material>
-        <sensor name="laser" type="ray">
-            <pose>0 0 0 0 0 0</pose>
-            <visualize>false</visualize>
-            <update_rate>10</update_rate>
-            <ray>
-                <scan>
-                    <horizontal>
-                        <samples>100</samples>
-                        <resolution>1.0</resolution>
-                        <min_angle>-1.22</min_angle>
-                        <max_angle>1.22</max_angle>
-                    </horizontal>
-                    <vertical>
-                        <samples>70</samples>
-                        <resolution>1.0</resolution>
-                        <min_angle>-0.3</min_angle>
-                        <max_angle>0.785</max_angle>
-                    </vertical>
-                </scan>
-                <range>
-                    <min>0.05</min>
-                    <max>5</max>
-                    <resolution>0.01</resolution>
-                </range>
-            </ray>
-            <plugin name="laser_scanner" filename="libgazebo_ros_ray_sensor.so">
-                <ros>
-                    <namespace>/</namespace>
-                    <argument>~/out:=scan</argument>
-                </ros>
-                <output_type>sensor_msgs/PointCloud2</output_type>
-                <frame_name>laser_3d_frame</frame_name>
-            </plugin>
-        </sensor>
-    </gazebo>
+    <xacro:include filename="uv_macros.xacro" />
+    <xacro:laser_sensor n="1" z="0.0" lower_angle="0.06" upper_angle="1.18" />
+    <!-- <xacro:laser_sensor n="2" z="0.3" lower_angle="1.03" upper_angle="1.36" /> -->
+    <xacro:laser_sensor n="3" z="0.6" lower_angle="0.9" upper_angle="0.9" />
+    <!-- <xacro:laser_sensor n="4" z="0.9" lower_angle="1.36" upper_angle="1.03" /> -->
+    <xacro:laser_sensor n="5" z="1.2" lower_angle="1.18" upper_angle="0.09" />
+    <!-- Pose ground truth publisher
+    <gazebo>
+        <plugin name="ground_truth" filename="libgazebo_ros_p3d.so">
+        <ros>
+            <namespace>/odometry</namespace>
+            <remapping>~/out:=ground_truth</remapping>
+        </ros>
+        <frame_name>map</frame_name>
+        <body_name>base_link</body_name>
+        <update_rate>50.0</update_rate>
+        </plugin>
+    </gazebo> -->
 </robot>

File: description/light.xacro (robot description, xacro)
@@ -5,5 +5,5 @@
         <parent link="chassis" />
         <child link="light_link" />
-        <origin xyz="${3/4 * length} 0 ${height + 0.5}" rpy="0 0 0" />
+        <origin xyz="${3/4 * length} 0 ${height + 0.6 + 0.05}" rpy="0 0 0" />
     </joint>
     <link name="light_link">
@@ -11,5 +11,5 @@
             <origin xyz="0 0 0" rpy="0 0 0" />
             <geometry>
-                <cylinder radius="0.02" length="1" />
+                <cylinder radius="0.01" length="1.2" />
             </geometry>
             <material name="white" />
@@ -18,5 +18,5 @@
             <origin xyz="0 0 0" rpy="0 0 0" />
             <geometry>
-                <cylinder radius="0.02" length="1" />
+                <cylinder radius="0.01" length="1.2" />
             </geometry>
         </collision>

Commit message: tuned params

File: description/lidar_3d.xacro (robot description, xacro)
@@ -2,9 +2,9 @@
 <robot xmlns:xacro="http://www.ros.org/wiki/xacro" name="robot">
     <xacro:include filename="uv_macros.xacro" />
-    <xacro:laser_sensor n="1" z="0.0" lower_angle="0.06" upper_angle="1.18" />
-    <!-- <xacro:laser_sensor n="2" z="0.3" lower_angle="1.03" upper_angle="1.36" /> -->
-    <xacro:laser_sensor n="3" z="0.6" lower_angle="0.9" upper_angle="0.9" />
-    <!-- <xacro:laser_sensor n="4" z="0.9" lower_angle="1.36" upper_angle="1.03" /> -->
-    <xacro:laser_sensor n="5" z="1.2" lower_angle="1.18" upper_angle="0.09" />
+    <xacro:laser_sensor n="1" z="0.0" lower_angle="0.15" upper_angle="1.41" />
+    <xacro:laser_sensor n="2" z="0.3" lower_angle="1.03" upper_angle="1.36" />
+    <xacro:laser_sensor n="3" z="0.6" lower_angle="1.26" upper_angle="1.26" />
+    <xacro:laser_sensor n="4" z="0.9" lower_angle="1.36" upper_angle="1.03" />
+    <xacro:laser_sensor n="5" z="1.2" lower_angle="1.41" upper_angle="0.15" />
     <!-- Pose ground truth publisher
     <gazebo>

File: description/uv_macros.xacro (robot description, xacro)
@@ -3,5 +3,5 @@
 <xacro:property name="uv_range" value="3" />
 <xacro:property name="horizontal_angle" value="2.46" />
-<xacro:property name="mesh_size" value="0.05" />
+<xacro:property name="mesh_size" value="0.1" />
 <xacro:macro name="laser_sensor" params="n z lower_angle upper_angle">
   <joint name="laser_3d_joint_${n}" type="fixed">
@@ -21,5 +21,5 @@
         <scan>
           <horizontal>
-            <samples>${round((uv_range * horizontal_angle) / mesh_size)}</samples>
+            <samples>${round((uv_range * horizontal_angle) / mesh_size) + 2}</samples>
             <resolution>1.0</resolution>
             <min_angle>-${horizontal_angle/2}</min_angle>
@@ -27,5 +27,5 @@
           </horizontal>
           <vertical>
-            <samples>${round((uv_range * (lower_angle + upper_angle)) / mesh_size)}</samples>
+            <samples>${round((uv_range * (lower_angle + upper_angle)) / mesh_size) + 2}</samples>
             <resolution>1.0</resolution>
             <min_angle>-${lower_angle}</min_angle>

Commit message: room uv

File: description/lidar_3d.xacro (robot description, xacro)
@@ -7,5 +7,5 @@
     <xacro:laser_sensor n="4" z="0.9" lower_angle="1.36" upper_angle="1.03" />
     <xacro:laser_sensor n="5" z="1.2" lower_angle="1.41" upper_angle="0.15" />
-    <!-- Pose ground truth publisher
+    <!-- Pose ground truth publisher  -->
     <gazebo>
         <plugin name="ground_truth" filename="libgazebo_ros_p3d.so">
@@ -16,6 +16,6 @@
         <frame_name>map</frame_name>
         <body_name>base_link</body_name>
-        <update_rate>50.0</update_rate>
+        <update_rate>1000.0</update_rate>
         </plugin>
-    </gazebo> -->
+    </gazebo>
 </robot>

File: description/uv_macros.xacro (robot description, xacro)
@@ -1,7 +1,7 @@
 <?xml version="1.0"?>
 <robot xmlns:xacro="http://www.ros.org/wiki/xacro" >
-<xacro:property name="uv_range" value="3" />
+<xacro:property name="uv_range" value="2" />
 <xacro:property name="horizontal_angle" value="2.46" />
-<xacro:property name="mesh_size" value="0.1" />
+<xacro:property name="mesh_size" value="0.05" />
 <xacro:macro name="laser_sensor" params="n z lower_angle upper_angle">
   <joint name="laser_3d_joint_${n}" type="fixed">

Commit message: lower base footprint

File: description/lidar_3d.xacro (robot description, xacro)
@@ -2,9 +2,16 @@
 <robot xmlns:xacro="http://www.ros.org/wiki/xacro" name="robot">
     <xacro:include filename="uv_macros.xacro" />
-    <xacro:laser_sensor n="1" z="0.0" lower_angle="0.15" upper_angle="1.41" />
+    <joint name="light_base_joint" type="fixed">
+        <parent link="chassis" />
+        <child link="light_base_link" />
+        <origin xyz="${3/4 * length} 0 ${height + 0.05}" rpy="0 0 0" />
+    </joint>
+    <link name="light_base_link">
+    </link>
+    <!-- <xacro:laser_sensor n="1" z="0.0" lower_angle="0.15" upper_angle="1.41" /> -->
     <!-- <xacro:laser_sensor n="2" z="0.3" lower_angle="1.03" upper_angle="1.36" /> -->
-    <xacro:laser_sensor n="3" z="0.6" lower_angle="1.26" upper_angle="1.26" />
+    <!-- <xacro:laser_sensor n="3" z="0.6" lower_angle="1.26" upper_angle="1.26" /> -->
     <!-- <xacro:laser_sensor n="4" z="0.9" lower_angle="1.36" upper_angle="1.03" /> -->
-    <xacro:laser_sensor n="5" z="1.2" lower_angle="1.41" upper_angle="0.15" />
+    <!-- <xacro:laser_sensor n="5" z="1.2" lower_angle="1.41" upper_angle="0.15" /> -->
     <!-- Pose ground truth publisher  -->
     <gazebo>

File: description/robot_core.xacro (robot description, xacro)
@@ -15,5 +15,5 @@
         <parent link="base_link"/>
         <child link="base_footprint"/>
-        <origin xyz="0 0 0" rpy="0 0 0"/>
+        <origin xyz="0 0 -${wheeldiam/2}" rpy="0 0 0"/>
     </joint>
     <link name="base_footprint">
